File: kicad_prototype/ELRS_ESP8285_PWM5_rev0.6.kicad_pcb (KiCad board)
At the start: 4 copper layers, 17.5 x 24.5 mm, 54 parts, among them J1 Conn_Coaxial, J2 Conn_01x05, J3 Conn_01x05, J4 Conn_01x05, J5 Conn_Coaxial, J6 Conn_01x02, U1 SPX3819M5-L-3-3, U2 ESP8285, U5 2450FM07D0034T, U6 SX1281, Y2 26M, Y3 52M

Commit message: general update
Parts:
- added C13: 10p, Capacitor_SMD:C_0402_1005Metric, F.Cu at (159.2, 68.4)
- D1: value LED -> blue_2V9
- D2: value LED -> true_gr_3V3
- D4: value LED -> red_2V1
- JP1: value SolderJumper_2_Bridged -> 4S; footprint Jumper:SolderJumper-2_P1.3mm_Bridged_RoundedPad1.0x1.5mm -> Jumper:SolderJumper-2_P1.3mm_Open_RoundedPad1.0x1.5mm
- R11: value 560R -> 270R
- R12: value 3k9 -> 4k7
- moved TP1 1.11 mm to (167.5, 60.1)
Connections:
- U2 pad 2: ANT -> Net-(C13-Pad2)
Routing:
- net ANT: track 17.8 -> 15.3 mm
- net Net-(C13-Pad2): track 0.00 -> 1.30 mm
Other:
- board text added: "1"
- board text added: "2 Tx"
- board text added: "3 Rx"
- board text added: "4"
- board text added: "4S"
- board text added: "5"
- board text added: "B"
- board text added: "GVS"
- board text added: "crteensy ELRS 8285 1280 PWM rev0.6"
- board text removed: "Boot"
- board text removed: "crteensy rev0.3"
